File: Hardware/PCB/timestamp generator Gen3 front panel/harp timestamp generator Gen3 front panel.kicad_pcb (KiCad board)
At the start: 2 copper layers, 133 x 35 mm, 12 parts

Commit message: Updated Gerbers.
Parts:
- added ref1: harp_logo, stepperdriver front panel:harp_logo, F.Cu at (93.6, 118.8)
Other:
- board text removed: "Powered by:"
